File: rcsdcard/v1/eagle/rcsdcard_v1.sch (EAGLE design)
At the start: 16 parts, among them IC1 74LS32N, IC2 74LS32N, IC3 74LS21N, IC4 74LS138N, IC5 74LS245N

Commit message: Add files via upload
Parts:
- added R1: 10k, rcl:R-EU_0204/7
Connections:
- net OE_L: now also R1.2
- net VCC: now also R1.1
Changed lines of the file:
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@@
 <part name="JP2" library="pinhead" library_urn="urn:adsk.eagle:library:325" deviceset="PINHD-1X20" device="" package3d_urn="urn:adsk.eagle:package:22441/2"/>
 <part name="JP4" library="pinhead" library_urn="urn:adsk.eagle:library:325" deviceset="PINHD-1X2" device="" package3d_urn="urn:adsk.eagle:package:22435/2"/>
+<part name="R1" library="rcl" library_urn="urn:adsk.eagle:library:334" deviceset="R-EU_" device="0204/7" package3d_urn="urn:adsk.eagle:package:23498/2" value="10k"/>
 </parts>
 <sheets>
@@
 <attribute name="VALUE" x="171.45" y="25.4" size="1.778" layer="96" rot="R180"/>
 </instance>
+<instance part="R1" gate="G$1" x="187.96" y="68.58" smashed="yes">
+<attribute name="NAME" x="184.15" y="70.0786" size="1.778" layer="95"/>
+<attribute name="VALUE" x="184.15" y="65.278" size="1.778" layer="96"/>
+</instance>
 </instances>
 <busses>
@@
 <pinref part="SUPPLY1" gate="G$1" pin="VCC"/>
 </segment>
+<segment>
+<pinref part="R1" gate="G$1" pin="1"/>
+<wire x1="182.88" y1="68.58" x2="177.8" y2="68.58" width="0.1524" layer="91"/>
+<label x="172.72" y="68.58" size="1.778" layer="95"/>
+</segment>
 </net>
 <net name="N$1" class="0">
@@
 <label x="238.76" y="66.04" size="1.778" layer="95"/>
 </segment>
-</net>
+<segment>
+<pinref part="R1" gate="G$1" pin="2"/>
+<wire x1="193.04" y1="68.58" x2="195.58" y2="68.58" width="0.1524" layer="91"/>
+<label x="198.12" y="68.58" size="1.778" layer="95"/>
+</segment>
+</net>
